File: sem_tanfolyampanel_2025.kicad_pcb (KiCad board)
At the start: 2 copper layers, 42.7 x 18 mm, 29 parts, among them J1 USB_C_Receptacle_USB2.0_16P, J2 Conn_01x09, J3 Conn_01x09, SW1 RESET, U1 STM32F030F4Px, U2 LD1117S33TR_SOT223, U3 CH32V203G6U6

Commit message: First iteration of PCB routing
Parts:
- removed TP1, TP2, TP3, TP4: TestPoint, TestPoint:TestPoint_Pad_D1.0mm
- added J4: PROG, jlcpcb:ProgConnector_5pin, B.Cu at (153.2, 58.8)
- BOOT: renamed from JP1; footprint Connector_PinHeader_2.54mm:PinHeader_2x01_P2.54mm_Vertical -> Jumper:SolderJumper-2_P1.3mm_Open_TrianglePad1.0x1.5mm
- moved R5 11.8 mm to (173.3, 60.7)
- moved C2 9.37 mm to (173.1, 51.2), turned to 0 degrees
- moved C3 8.67 mm to (161.9, 60.1), turned to 180 degrees
- moved C1 6.78 mm to (165.0, 60.1), turned to 180 degrees
- moved U2 3.41 mm to (163.4, 54.7), turned to 90 degrees
- moved R7 3.00 mm to (157.2, 59.6)
- moved BOOT 1.39 mm to (155.8, 50.1), turned to 90 degrees
- moved R6 0.54 mm to (158.8, 59.6), turned to -90 degrees
- moved R2 0.36 mm to (176.6, 51.2)
- moved R3 0.26 mm to (151.6, 51.2), turned to -90 degrees
- moved C4 0.13 mm to (159.0, 54.2)
Connections:
- net Net-(U3-~{RST}) renamed /P_nRST
- U3 pad 21: Net-(U3-PA13/SWDIO) -> /P_SWD
- U3 pad 22: Net-(U3-PA14/SWCLK) -> /P_SWC
Routing:
- net /NRST: track 0.00 -> 51.2 mm, vias 0 -> 2
- net +3V3: track 7.20 -> 57.1 mm, vias 0 -> 3
- net /UART_RX: track 0.00 -> 31.5 mm, vias 0 -> 2
- net /UART_TX: track 0.00 -> 30.5 mm, vias 0 -> 2
- net Net-(JP1-A): track 0.00 -> 15.1 mm
- net /SWDIO: track 0.00 -> 14.7 mm, vias 0 -> 2
- net /SWCLK: track 0.00 -> 13.9 mm, vias 0 -> 2
- net /PF0: track 0.00 -> 13.6 mm, vias 0 -> 1
- net /PA10: track 0.00 -> 11.6 mm, vias 0 -> 1
- net +5V: track 11.1 -> 21.9 mm
- net /PF1: track 0.00 -> 10.6 mm, vias 0 -> 1
- net /PA0: track 0.00 -> 9.89 mm, vias 0 -> 1
- net /PA9: track 0.00 -> 9.74 mm, vias 0 -> 1
- net /PB1: track 0.00 -> 9.50 mm, vias 0 -> 1
- net /P_nRST: track 0.00 -> 7.89 mm, vias 0 -> 1
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Other:
- board text added: "UART TX:PA2 RX:PA3"
- board text removed: "UART TX:PA2, RX:PA3"

Commit message: Rerouting and finalizing.
Parts:
- removed BOOT: Programmer boot, Jumper:SolderJumper-2_P1.3mm_Open_TrianglePad1.0x1.5mm
- added JP1: Programmer boot, Jumper:SolderJumper-2_P1.3mm_Open_TrianglePad1.0x1.5mm, F.Cu at (155.7, 49.5)
- C1, C3: footprint Capacitor_SMD:C_0603_1608Metric -> Capacitor_SMD:C_0805_2012Metric
- moved D2 8.29 mm to (177.9, 56.1), turned to 90 degrees
- moved R7 3.40 mm to (160.6, 59.6)
- moved C1 2.94 mm to (167.9, 60.4), turned to 0 degrees
- moved U2 2.44 mm to (165.9, 54.9)
- moved C5 2.08 mm to (153.9, 53.1)
- moved C4 2.05 mm to (160.9, 53.4)
- moved U3 2.02 mm to (157.4, 54.4)
- moved C3 1.97 mm to (163.9, 60.4)
- moved J4 1.04 mm to (154.2, 58.8)
- moved F1 0.94 mm to (153.4, 62.9)
- moved R4 0.52 mm to (152.1, 58.4)
- moved R3 0.51 mm to (152.1, 51.4), turned to 90 degrees
- moved R5 0.42 mm to (172.9, 60.6)
- moved C2 0.29 mm to (173.4, 51.1)
- moved R2 0.29 mm to (176.9, 51.1)
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Connections:
- J1 pad A8: Net-(J1-SBU1) -> unconnected-(J1-SBU1-PadA8)
- J1 pad B8: Net-(J1-SBU2) -> unconnected-(J1-SBU2-PadB8)
- U3 pad 29: (no net) -> GND
Routing:
- net GND: track 2.74 -> 51.1 mm, vias 23 -> 68
- net +3V3: track 57.1 -> 72.7 mm, vias 3 -> 4
- net Net-(F1-Pad1): track 11.9 -> 22.0 mm, vias 3 -> 2
- net /UART_RX: track 31.5 -> 25.3 mm, vias 2 -> 1
- net /PB1: track 9.50 -> 14.9 mm
- net /NRST: track 51.2 -> 46.8 mm, vias 2 -> 3
- net Net-(J1-CC1): track 7.35 -> 4.19 mm, vias 2 -> 0
- net /USBD_N: track 6.30 -> 8.59 mm
- net /UART_TX: track 30.5 -> 28.4 mm
- net /P_nRST: track 7.89 -> 9.81 mm, vias 1 -> 0
- net /P_SWD: track 5.03 -> 6.69 mm, vias 1 -> 0
- net /P_SWC: track 2.23 -> 3.82 mm
- net /SWCLK: track 13.9 -> 15.4 mm
- net /PF1: track 10.6 -> 11.8 mm
- net /PA1: track 7.82 -> 6.71 mm
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Other:
- board size 42.7 x 18 mm -> 43 x 18 mm
- board text added: "+3V3"
- board text added: "+5V"
- board text added: "Elkövetők: W.P. & H.K."
- board text added: "GND"
- board text added: "PA0"
- board text added: "PA1"
- board text added: "PA10"
- board text added: "PA2"
- board text added: "PA3"
- board text added: "PA4"
- board text added: "PA5"
- board text added: "PA6"
- board text added: "PA7"
- board text added: "PA9"
- board text added: "PB1"
- board text added: "PF0"
- board text added: "PF1"
- board text added: "PRG"
- board text added: "nRST"
- board text removed: "COM"
- board text removed: "Elkövető: W.P."
