File: hardware/sem_tanfolyampanel_2025.kicad_pcb (KiCad board)
At the start: 2 copper layers, 43 x 18 mm, 26 parts, among them J1 USB_C_Receptacle_USB2.0_16P, J2 Conn_01x09, J3 Conn_01x09, J4 PROG, SW1 RESET, U1 STM32F030F4Px, U2 LD1117S33TR_SOT223, U3 CH32V203G6U6

Commit message: Rev.A1
Parts:
- removed JP1: Programmer boot, Jumper:SolderJumper-2_P1.3mm_Open_TrianglePad1.0x1.5mm
- added TP1: Programmer boot, TestPoint:TestPoint_THTPad_D1.5mm_Drill0.7mm, F.Cu at (157.0, 49.8)
Routing:
- net Net-(U3-BOOT0/PB8): track 15.2 -> 13.2 mm, vias 2 -> 1
- net +3V3: track 72.7 -> 71.7 mm
Other:
- board text added: "Boot"
- board text added: "Rev.A1"
- board text added: "UART TX: PA2 RX: PA3"
- board text added: "Vesztettem"
- board text removed: "Rev.A"
- board text removed: "UART TX:PA2 RX:PA3"
