File: hardware/sem_tanfolyampanel_2025.kicad_sch (KiCad schematic)
At the start: 26 parts, among them J1 USB_C_Receptacle_USB2.0_16P, J2 Conn_01x09, J3 Conn_01x09, J4 PROG, SW1 RESET, U1 STM32F030F4Px, U2 LD1117S33TR_SOT223, U3 CH32V203G6U6

Commit message: Rev.A1
Parts:
- removed JP1: Programmer boot, Jumper:SolderJumper-2_P1.3mm_Open_TrianglePad1.0x1.5mm, symbol Jumper:Jumper_2_Open
- added TP1: Programmer boot, TestPoint:TestPoint_THTPad_D1.5mm_Drill0.7mm, symbol Connector:TestPoint
Connections:
- net at R6.1, U3.1 (BOOT0/PB8): now also TP1.1

Commit message: Sent to fab.
Other:
- company: Weisz Pál -> Weisz Pál, Horváth Kristóf
- title: One dollar ARM devboard -> SEM tanfolyam panel 2025
Changed lines of the file:
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@@
 	(paper "A4")
 	(title_block
-		(title "One dollar ARM devboard")
-		(date "2024-11-19")
+		(title "SEM tanfolyam panel 2025")
+		(date "2025-01-16")
 		(rev "C")
-		(company "Weisz Pál")
+		(company "Weisz Pál, Horváth Kristóf")
 	)
 	(junction
